File: levelConversionOpAmp/levelConversionOpAmp.sch (KiCad schematic (older format))
At the start: 12 parts, among them J1 IN, J2 OUT, J3 POW, U1 TL082

Commit message: Placement des composantes sur plaque perforee
Connections:
- net GND: now also J2.2 (Pin_2); no longer J2.1 (Pin_1)
- net SIGOUT: now also J2.1 (Pin_1); no longer J2.2 (Pin_2)
Changed lines of the file:
@@
 Wire Wire Line
 	5100 3300 5850 3300
-$Comp
-L Connector:Conn_01x02_Female J2
-U 1 1 6463C2CC
-P 8700 4200
-F 0 "J2" V 8546 4248 50  0000 L CNN
-F 1 " OUT" V 8637 4248 50  0000 L CNN
-F 2 "TerminalBlock:TerminalBlock_Altech_AK300-2_P5.00mm" H 8700 4200 50  0001 C CNN
-F 3 "~" H 8700 4200 50  0001 C CNN
-	1    8700 4200
-	0    1    1    0
-$EndComp
 Wire Wire Line
 	8400 3700 8600 3700
@@
 Wire Wire Line
 	9650 4050 9650 4000
-Wire Wire Line
-	9650 4000 8700 4000
 Wire Wire Line
 	7550 3700 8100 3700
@@
 	1550 3400 2050 3400
 Connection ~ 2050 3400
+$Comp
+L Connector:Conn_01x02_Female J2
+U 1 1 6463C2CC
+P 8600 4200
+F 0 "J2" V 8446 4248 50  0000 L CNN
+F 1 " OUT" V 8537 4248 50  0000 L CNN
+F 2 "TerminalBlock:TerminalBlock_Altech_AK300-2_P5.00mm" H 8600 4200 50  0001 C CNN
+F 3 "~" H 8600 4200 50  0001 C CNN
+	1    8600 4200
+	0    -1   1    0
+$EndComp
+Wire Wire Line
+	8700 4000 9650 4000
 $EndSCHEMATC

Commit message: Changed layout a little. Added ground bias resistor at output to quickly set output DC level even when plugged into a high impedance load
Parts:
- added R9: 4k7, Resistor_THT:R_Axial_DIN0207_L6.3mm_D2.5mm_P7.62mm_Horizontal, symbol Device:R_Small_US
Connections:
- net GND: now also R9.1
- net SIGOUT: now also R9.2
Changed lines of the file:
@@
 	8600 3700 8600 4000
 Wire Wire Line
-	8600 3700 8900 3700
+	8600 3700 8800 3700
 Connection ~ 8600 3700
 $Comp
@@
 $EndComp
 Wire Wire Line
-	8700 4000 9650 4000
+	8700 4000 8800 4000
+$Comp
+L Device:R_Small_US R9
+U 1 1 64905615
+P 8800 3850
+F 0 "R9" V 8595 3850 50  0000 C CNN
+F 1 "4k7" V 8686 3850 50  0000 C CNN
+F 2 "Resistor_THT:R_Axial_DIN0207_L6.3mm_D2.5mm_P7.62mm_Horizontal" H 8800 3850 50  0001 C CNN
+F 3 "~" H 8800 3850 50  0001 C CNN
+	1    8800 3850
+	-1   0    0    1
+$EndComp
+Wire Wire Line
+	8800 3700 8800 3750
+Connection ~ 8800 3700
+Wire Wire Line
+	8800 3700 8900 3700
+Wire Wire Line
+	8800 3950 8800 4000
+Connection ~ 8800 4000
+Wire Wire Line
+	8800 4000 9650 4000
 $EndSCHEMATC
